File: add.kicad_pcb (KiCad board)
At the start: 2 copper layers, 35.1 x 89.7 mm, 36 parts, among them J1 Conn_02x05_Odd_Even, J2 in0, J3 in1, J4 in2, J5 out, J6 Conn_01x03_Pin, J7 Conn_01x03_Socket, J8 Conn_01x03_Pin, J9 Conn_01x03_Socket, U1 TL072

Commit message: update bom for sync
Parts:
- C3: value C -> 100u
- J6, J8: footprint Connector_PinSocket_2.54mm:PinSocket_1x03_P2.54mm_Vertical -> Connector_PinHeader_2.54mm:PinHeader_1x03_P2.54mm_Vertical
Changed lines of the file:
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@@
 			)
 		)
-		(property "Value" "C"
+		(property "Value" "100u"
 			(at 0 1.68 0)
 			(layer "F.Fab")
@@
 		(sheetname "/")
 		(sheetfile "add.kicad_sch")
+		(units
+			(unit
+				(name "A")
+				(pins "1")
+			)
+		)
 		(attr through_hole exclude_from_bom)
 		(duplicate_pad_numbers_are_jumpers no)
@@
 		(sheetname "/")
 		(sheetfile "add.kicad_sch")
+		(units
+			(unit
+				(name "A")
+				(pins "1")
+			)
+		)
 		(attr through_hole exclude_from_bom)
 		(duplicate_pad_numbers_are_jumpers no)
@@
 		(sheetname "/")
 		(sheetfile "add.kicad_sch")
+		(units
+			(unit
+				(name "A")
+				(pins "1")
+			)
+		)
 		(attr through_hole exclude_from_bom)
 		(duplicate_pad_numbers_are_jumpers no)
@@
 		(sheetname "/")
 		(sheetfile "add.kicad_sch")
+		(units
+			(unit
+				(name "A")
+				(pins "1")
+			)
+		)
 		(attr through_hole exclude_from_bom)
 		(duplicate_pad_numbers_are_jumpers no)
@@
 		)
 	)
-	(footprint "Connector_PinSocket_2.54mm:PinSocket_1x03_P2.54mm_Vertical"
+	(footprint "Connector_PinHeader_2.54mm:PinHeader_1x03_P2.54mm_Vertical"
 		(layer "B.Cu")
 		(at 89.916 83.312)
-		(descr "Through hole straight socket strip, 1x03, 2.54mm pitch, single row (from Kicad 4.0.7), script generated")
-		(tags "Through hole socket strip THT 1x03 2.54mm single row")
+		(descr "Through hole straight pin header, 1x03, 2.54mm pitch, single row")
+		(tags "Through hole pin header THT 1x03 2.54mm single row")
 		(property "Reference" "J6"
-			(at 0 2.77 0)
+			(at 0 2.33 180)
 			(layer "B.SilkS")
 			(effects
@@
 		)
 		(property "Value" "Conn_01x03_Pin"
-			(at 0 -7.85 0)
+			(at 0 -7.41 180)
 			(layer "B.Fab")
 			(effects
@@
 		)
 		(property "Datasheet" ""
-			(at 0 0 0)
+			(at 0 0 180)
 			(layer "B.Fab")
 			(hide yes)
@@
 		)
 		(property "Description" "Generic connector, single row, 01x03, script generated"
-			(at 0 0 0)
+			(at 0 0 180)
 			(layer "B.Fab")
 			(hide yes)
@@
 		)
 		(fp_line
-			(start 0 1.33)
-			(end 1.33 1.33)
+			(start -1.33 0)
+			(end -1.33 1.33)
 			(stroke
 				(width 0.12)
@@
 		)
 		(fp_line
-			(start 1.33 -1.27)
-			(end 1.33 -6.41)
+			(start -1.33 1.33)
+			(end 0 1.33)
 			(stroke
 				(width 0.12)
@@
 		)
 		(fp_line
-			(start 1.33 1.33)
-			(end 1.33 0)
+			(start 1.33 -1.27)
+			(end 1.33 -6.41)
 			(stroke
 				(width 0.12)
@@
 		(fp_line
 			(start -1.8 -6.85)
-			(end -1.8 1.8)
+			(end 1.8 -6.85)
 			(stroke
 				(width 0.05)
@@
 		(fp_line
 			(start -1.8 1.8)
-			(end 1.75 1.8)
+			(end -1.8 -6.85)
 			(stroke
 				(width 0.05)
@@
 		)
 		(fp_line
-			(start 1.75 -6.85)
-			(end -1.8 -6.85)
+			(start 1.8 -6.85)
+			(end 1.8 1.8)
 			(stroke
 				(width 0.05)
@@
 		)
 		(fp_line
-			(start 1.75 1.8)
-			(end 1.75 -6.85)
+			(start 1.8 1.8)
+			(end -1.8 1.8)
 			(stroke
 				(width 0.05)
@@
 		(fp_line
 			(start -1.27 -6.35)
-			(end -1.27 1.27)
+			(end -1.27 0.635)
 			(stroke
 				(width 0.1)
@@
 		)
 		(fp_line
-			(start -1.27 1.27)
-			(end 0.635 1.27)
+			(start -1.27 0.635)
+			(end -0.635 1.27)
 			(stroke
 				(width 0.1)
@@
 		)
 		(fp_line
-			(start 0.635 1.27)
-			(end 1.27 0.635)
+			(start -0.635 1.27)
+			(end 1.27 1.27)
 			(stroke
 				(width 0.1)
@@
 		)
 		(fp_line
-			(start 1.27 0.635)
+			(start 1.27 1.27)
 			(end 1.27 -6.35)
 			(stroke
@@
 		)
 		(embedded_fonts no)
-		(model "${KICAD6_3DMODEL_DIR}/Connector_PinSocket_2.54mm.3dshapes/PinSocket_1x03_P2.54mm_Vertical.wrl"
+		(model "${KICAD6_3DMODEL_DIR}/Connector_PinHeader_2.54mm.3dshapes/PinHeader_1x03_P2.54mm_Vertical.wrl"
 			(offset
 				(xyz 0 0 0)
@@
 		)
 	)
-	(footprint "Connector_PinSocket_2.54mm:PinSocket_1x03_P2.54mm_Vertical"
+	(footprint "Connector_PinHeader_2.54mm:PinHeader_1x03_P2.54mm_Vertical"
 		(layer "B.Cu")
 		(at 59.944 90.932 180)
-		(descr "Through hole straight socket strip, 1x03, 2.54mm pitch, single row (from Kicad 4.0.7), script generated")
-		(tags "Through hole socket strip THT 1x03 2.54mm single row")
+		(descr "Through hole straight pin header, 1x03, 2.54mm pitch, single row")
+		(tags "Through hole pin header THT 1x03 2.54mm single row")
 		(property "Reference" "J8"
-			(at -2.5146 1.1176 0)
+			(at 0 2.33 0)
 			(layer "B.SilkS")
 			(effects
@@
 		)
 		(property "Value" "Conn_01x03_Pin"
-			(at 0 -7.85 0)
+			(at 0 -7.41 0)
 			(layer "B.Fab")
 			(effects
@@
 		(duplicate_pad_numbers_are_jumpers no)
 		(fp_line
-			(start 1.33 1.33)
-			(end 1.33 0)
+			(start 1.33 -1.27)
+			(end 1.33 -6.41)
 			(stroke
 				(width 0.12)
@@
 		)
 		(fp_line
-			(start 1.33 -1.27)
-			(end 1.33 -6.41)
+			(start -1.33 1.33)
+			(end 0 1.33)
 			(stroke
 				(width 0.12)
@@
 		)
 		(fp_line
-			(start 0 1.33)
-			(end 1.33 1.33)
+			(start -1.33 0)
+			(end -1.33 1.33)
 			(stroke
 				(width 0.12)
@@
 		)
 		(fp_line
-			(start 1.75 1.8)
-			(end 1.75 -6.85)
+			(start 1.8 1.8)
+			(end -1.8 1.8)
 			(stroke
 				(width 0.05)
@@
 		)
 		(fp_line
-			(start 1.75 -6.85)
-			(end -1.8 -6.85)
+			(start 1.8 -6.85)
+			(end 1.8 1.8)
 			(stroke
 				(width 0.05)
@@
 		(fp_line
 			(start -1.8 1.8)
-			(end 1.75 1.8)
+			(end -1.8 -6.85)
 			(stroke
 				(width 0.05)
@@
 		(fp_line
 			(start -1.8 -6.85)
-			(end -1.8 1.8)
+			(end 1.8 -6.85)
 			(stroke
 				(width 0.05)
@@
 		)
 		(fp_line
-			(start 1.27 0.635)
+			(start 1.27 1.27)
 			(end 1.27 -6.35)
 			(stroke
@@
 		)
 		(fp_line
-			(start 0.635 1.27)
-			(end 1.27 0.635)
+			(start -0.635 1.27)
+			(end 1.27 1.27)
 			(stroke
 				(width 0.1)
@@
 		)
 		(fp_line
-			(start -1.27 1.27)
-			(end 0.635 1.27)
+			(start -1.27 0.635)
+			(end -0.635 1.27)
 			(stroke
 				(width 0.1)
@@
 		(fp_line
 			(start -1.27 -6.35)
-			(end -1.27 1.27)
+			(end -1.27 0.635)
 			(stroke
 				(width 0.1)
@@
 		)
 		(fp_text user "${REFERENCE}"
-			(at 0 -2.54 90)
+			(at 0 -2.54 270)
 			(layer "B.Fab")
 			(effects
@@
 		)
 		(embedded_fonts no)
-		(model "${KICAD6_3DMODEL_DIR}/Connector_PinSocket_2.54mm.3dshapes/PinSocket_1x03_P2.54mm_Vertical.wrl"
+		(model "${KICAD6_3DMODEL_DIR}/Connector_PinHeader_2.54mm.3dshapes/PinHeader_1x03_P2.54mm_Vertical.wrl"
 			(offset
 				(xyz 0 0 0)

Commit message: fix capacitor value
Parts:
- C3: value 100u -> 100n
Changed lines of the file:
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@@
 			)
 		)
-		(property "Value" "100u"
+		(property "Value" "100n"
 			(at 0 1.68 0)
 			(layer "F.Fab")

Commit message: normal inputs to ground
Connections:
- J2 pad TN: unconnected-(J2-PadTN) -> /GND'
- J3 pad TN: unconnected-(J3-PadTN) -> /GND'
- J4 pad TN: unconnected-(J4-PadTN) -> /GND'
Changed lines of the file:
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@@
 			(layers "*.Cu" "*.Mask")
 			(remove_unused_layers no)
-			(net "unconnected-(J4-PadTN)")
-			(pintype "passive+no_connect")
+			(net "/GND'")
+			(pintype "passive")
 		)
 		(embedded_fonts no)
@@
 			(layers "*.Cu" "*.Mask")
 			(remove_unused_layers no)
-			(net "unconnected-(J3-PadTN)")
-			(pintype "passive+no_connect")
+			(net "/GND'")
+			(pintype "passive")
 		)
 		(embedded_fonts no)
@@
 			(layers "*.Cu" "*.Mask")
 			(remove_unused_layers no)
-			(net "unconnected-(J2-PadTN)")
-			(pintype "passive+no_connect")
+			(net "/GND'")
+			(pintype "passive")
 		)
 		(embedded_fonts no)
