File: add.kicad_sch (KiCad schematic)
At the start: 42 parts, among them J1 Conn_02x05_Odd_Even, J2 in0, J3 in1, J4 in2, J5 out, J6 Conn_01x03_Pin, J7 Conn_01x03_Socket, J8 Conn_01x03_Pin, J9 Conn_01x03_Socket, M1 Standoff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

Commit message: update bom for sync
Parts:
- C3: value C -> 100u
- J6, J8: footprint Connector_PinSocket_2.54mm:PinSocket_1x03_P2.54mm_Vertical -> Connector_PinHeader_2.54mm:PinHeader_1x03_P2.54mm_Vertical
Other:
- moved on the sheet: C3
Changed lines of the file:
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@@
 	(wire
 		(pts
-			(xy 97.79 92.71) (xy 97.79 96.52)
+			(xy 95.25 92.71) (xy 95.25 96.52)
 		)
 		(stroke
@@
 	(wire
 		(pts
-			(xy 102.87 92.71) (xy 97.79 92.71)
+			(xy 102.87 92.71) (xy 95.25 92.71)
 		)
 		(stroke
@@
 	(wire
 		(pts
-			(xy 97.79 107.95) (xy 97.79 104.14)
+			(xy 95.25 107.95) (xy 95.25 104.14)
 		)
 		(stroke
@@
 	(wire
 		(pts
-			(xy 102.87 107.95) (xy 97.79 107.95)
+			(xy 102.87 107.95) (xy 95.25 107.95)
 		)
 		(stroke
@@
 	(symbol
 		(lib_id "Device:C")
-		(at 97.79 100.33 0)
+		(at 95.25 100.33 0)
 		(unit 1)
 		(body_style 1)
@@
 		(fields_autoplaced yes)
 		(property "Reference" "C3"
-			(at 101.6 99.0599 0)
+			(at 99.06 99.0599 0)
 			(show_name no)
 			(do_not_autoplace no)
@@
 			)
 		)
-		(property "Value" "C"
-			(at 101.6 101.5999 0)
+		(property "Value" "100u"
+			(at 99.06 101.5999 0)
 			(show_name no)
 			(do_not_autoplace no)
@@
 		)
 		(property "Footprint" "Capacitor_SMD:C_0805_2012Metric"
-			(at 98.7552 104.14 0)
+			(at 96.2152 104.14 0)
 			(hide yes)
 			(show_name no)
@@
 		)
 		(property "Datasheet" ""
-			(at 97.79 100.33 0)
+			(at 95.25 100.33 0)
 			(hide yes)
 			(show_name no)
@@
 		)
 		(property "Description" "Unpolarized capacitor"
-			(at 97.79 100.33 0)
+			(at 95.25 100.33 0)
 			(hide yes)
 			(show_name no)
@@
 			)
 		)
-		(property "Footprint" "Connector_PinSocket_2.54mm:PinSocket_1x03_P2.54mm_Vertical"
+		(property "Footprint" "Connector_PinHeader_2.54mm:PinHeader_1x03_P2.54mm_Vertical"
 			(at 41.91 119.38 0)
 			(hide yes)
@@
 			)
 		)
-		(property "Footprint" "Connector_PinSocket_2.54mm:PinSocket_1x03_P2.54mm_Vertical"
+		(property "Footprint" "Connector_PinHeader_2.54mm:PinHeader_1x03_P2.54mm_Vertical"
 			(at 41.91 105.41 0)
 			(hide yes)

Commit message: fix capacitor value
Parts:
- C3: value 100u -> 100n
Changed lines of the file:
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@@
 			)
 		)
-		(property "Value" "100u"
+		(property "Value" "100n"
 			(at 99.06 101.5999 0)
 			(show_name no)

Commit message: normal inputs to ground
Connections:
- net GND': now also J2.TN, J3.TN, J4.TN
- no-connect marks 4 -> 1
Changed lines of the file:
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@@
-	)
-	(no_connect
-		(at 40.64 66.04)
 	)
 	(no_connect
 		(at 40.64 82.55)
 	)
-	(no_connect
-		(at 40.64 33.02)
-	)
-	(no_connect
-		(at 40.64 49.53)
-	)
 	(wire
 		(pts
@@
 		)
 	)
+	(label "GND'"
+		(at 40.64 49.53 0)
+		(effects
+			(font
+				(size 1.27 1.27)
+			)
+			(justify left bottom)
+		)
+	)
 	(label "FACE"
 		(at 16.51 187.96 0)
@@
 		)
 	)
+	(label "GND'"
+		(at 40.64 33.02 0)
+		(effects
+			(font
+				(size 1.27 1.27)
+			)
+			(justify left bottom)
+		)
+	)
+	(label "GND'"
+		(at 40.64 66.04 0)
+		(effects
+			(font
+				(size 1.27 1.27)
+			)
+			(justify left bottom)
+		)
+	)
